File: Boards/First/First.kicad_pcb (KiCad board)
At the start: 2 copper layers, 100 x 100 mm, 148 parts, among them J1 Conn_02x10_Odd_Even, J4 Conn_02x19_Odd_Even, J5 Barrel_Jack, K1 Relay_SPDT, K10 Relay_SPDT, K11 Relay_SPDT, K12 Relay_SPDT, K13 Relay_SPDT, K14 Relay_SPDT, K15 Relay_SPDT, K16 Relay_SPDT, K17 Relay_SPDT, K18 Relay_SPDT, K19 Relay_SPDT, K2 Relay_SPDT, K20 Relay_SPDT, K21 Relay_SPDT, K22 Relay_SPDT, K23 Relay_SPDT, K24 Relay_SPDT, K25 Relay_SPDT, K26 Relay_SPDT, K27 Relay_SPDT, K28 Relay_SPDT, K29 Relay_SPDT, K3 Relay_SPDT, K30 Relay_SPDT, K31 Relay_SPDT, K32 Relay_SPDT, K33 Relay_SPDT, K34 Relay_SPDT, K35 Relay_SPDT, K36 Relay_SPDT, K4 Relay_SPDT, K5 Relay_SPDT, K6 Relay_SPDT, K7 Relay_SPDT, K8 Relay_SPDT, K9 Relay_SPDT

Commit message: general
Routing:
- net /S2S0: track 155.1 -> 153.7 mm
- net GND: vias 30 -> 31
Changed lines of the file:
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@@
 	)
 	(via
+		(at 126.5 84)
+		(size 0.5)
+		(drill 0.3)
+		(layers "F.Cu" "B.Cu")
+		(free yes)
+		(net "GND")
+	)
+	(via
 		(at 53.5 119)
 		(size 0.8)
@@
 	)
 	(segment
+		(start 72.5 106.118309)
+		(end 72.5 99.08941)
+		(width 0.2)
+		(layer "F.Cu")
+		(net "/S4S0")
+	)
+	(segment
 		(start 64.052715 126)
 		(end 68 126)
@@
 	)
 	(segment
-		(start 72.5 106.5)
-		(end 72.5 99.08941)
-		(width 0.2)
-		(layer "F.Cu")
-		(net "/S4S0")
-	)
-	(segment
 		(start 61.81 128.242715)
 		(end 64.052715 126)
@@
 	)
 	(segment
+		(start 72.626667 106.244976)
+		(end 72.5 106.118309)
+		(width 0.2)
+		(layer "F.Cu")
+		(net "/S4S0")
+	)
+	(segment
 		(start 86.92125 67.7925)
 		(end 82.913483 67.7925)
@@
 	)
 	(via
-		(at 72.5 106.5)
+		(at 72.626667 106.244976)
 		(size 0.6)
 		(drill 0.3)
@@
 	)
 	(segment
+		(start 72.626667 106.373333)
+		(end 71.5 107.5)
+		(width 0.2)
+		(layer "B.Cu")
+		(net "/S4S0")
+	)
+	(segment
+		(start 71.5 107.5)
+		(end 71.5 111)
+		(width 0.2)
+		(layer "B.Cu")
+		(net "/S4S0")
+	)
+	(segment
 		(start 75.657498 74.5)
 		(end 76.5 73.657498)
@@
 	)
 	(segment
-		(start 71.5 111)
-		(end 71.5 107.5)
-		(width 0.2)
-		(layer "B.Cu")
-		(net "/S4S0")
-	)
-	(segment
 		(start 69.5475 93)
 		(end 70 93)
@@
 	)
 	(segment
-		(start 68 126)
-		(end 68 125.5)
+		(start 72.626667 106.244976)
+		(end 72.626667 106.373333)
 		(width 0.2)
 		(layer "B.Cu")
@@
 	)
 	(segment
-		(start 71.5 107.5)
-		(end 72.5 106.5)
+		(start 68 126)
+		(end 68 125.5)
 		(width 0.2)
 		(layer "B.Cu")
@@
 	)
 	(segment
+		(start 68.430295 110.222793)
+		(end 66.890957 110.222793)
+		(width 0.2)
+		(layer "F.Cu")
+		(net "/S2S0")
+	)
+	(segment
+		(start 51.41 127.741471)
+		(end 51.41 130.35)
+		(width 0.2)
+		(layer "F.Cu")
+		(net "/S2S0")
+	)
+	(segment
 		(start 51.41 130.35)
 		(end 50.26 131.5)
@@
 	)
 	(segment
-		(start 68.430295 110.222793)
-		(end 66.890957 110.222793)
+		(start 53.751471 125.4)
+		(end 51.41 127.741471)
 		(width 0.2)
 		(layer "F.Cu")
@@
 	)
 	(segment
-		(start 61.824284 125.4)
-		(end 51.41 125.4)
-		(width 0.2)
-		(layer "F.Cu")
-		(net "/S2S0")
-	)
-	(segment
 		(start 103.00125 54.3325)
 		(end 103.00125 55.746713)
@@
 	)
 	(segment
-		(start 51.41 125.4)
-		(end 51.41 130.35)
+		(start 61.824284 125.4)
+		(end 53.751471 125.4)
 		(width 0.2)
 		(layer "F.Cu")
