File: Boards/interfaceBoard/interfaceBoard/_restore_backup_2026-09-19T00-12-02-279/output.kicad_sch (KiCad schematic)
At the start: 2 parts, among them U1 74HC595, U2 TBD62783A

Commit message: interface board work
finished the MOSI child sheet
finished the MISO child sheet
started work on pcb layout (only 1 MOSI and MISO)
started work on pcb layout
Parts:
- removed U2: TBD62783A, Package_DIP:DIP-18_W7.62mm_Socket, symbol Transistor_Array:TBD62783A
- U1: footprint Package_DIP:DIP-16_W7.62mm_Socket -> (none)
Connections:
- net 5V+ renamed VCC
- net SerIn renamed MOSI
Other:
- note removed: "Index on output from shift reg and input to power controll swapped as this better matches the pinout of the actual ICs"
