File: Boards/interfaceBoard/interfaceBoard/MISO_sheet.kicad_sch (KiCad schematic)
At the start: 1 part, among them U3 74HC165

Commit message: Big progress
Parts:
- added RN1: R_Pack08, Package_DIP:DIP-16_W7.62mm_Socket, symbol Device:R_Pack08
- added RN2: R_Network08, Resistor_THT:R_Array_SIP9, symbol Device:R_Network08
Connections:
- net D0: now also RN1.9 (R8.2)
- net D1: now also RN1.10 (R7.2)
- net D2: now also RN1.11 (R6.2)
- net D3: now also RN1.12 (R5.2)
- net D4: now also RN1.13 (R4.2)
- net D5: now also RN1.14 (R3.2)
- net D6: now also RN1.15 (R2.2)
- net D7: now also RN1.16 (R1.2)
- net GND: now also RN2.1 (common)
- net vDiv0/OUT: no longer names the net of U3.11 (D0)
- net vDiv0/OUT: now also RN1.8 (R8.1), RN2.9 (R8)
- net vDiv1/OUT: no longer names the net of U3.12 (D1)
- net vDiv1/OUT: now also RN1.7 (R7.1), RN2.8 (R7)
- net vDiv2/OUT: no longer names the net of U3.13 (D2)
- net vDiv2/OUT: now also RN1.6 (R6.1), RN2.7 (R6)
- net vDiv3/OUT: no longer names the net of U3.14 (D3)
- net vDiv3/OUT: now also RN1.5 (R5.1), RN2.6 (R5)
- net vDiv4/OUT: no longer names the net of U3.3 (D4)
- net vDiv4/OUT: now also RN1.4 (R4.1), RN2.5 (R4)
- net vDiv5/OUT: no longer names the net of U3.4 (D5)
- net vDiv5/OUT: now also RN1.3 (R3.1), RN2.4 (R3)
- net vDiv6/OUT: no longer names the net of U3.5 (D6)
- net vDiv6/OUT: now also RN1.2 (R2.1), RN2.3 (R2)
- net vDiv7/OUT: no longer names the net of U3.6 (D7)
- net vDiv7/OUT: now also RN1.1 (R1.1), RN2.2 (R1)
Other:
- removed sheet vDiv0
- removed sheet vDiv1
- removed sheet vDiv2
- removed sheet vDiv3
- removed sheet vDiv4
- removed sheet vDiv5
- removed sheet vDiv6
- removed sheet vDiv7

Commit message: MOSI done?
MOSI wired.
MISO wired to interface
Changed lines of the file:
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@@
 		(dnp no)
 		(property "Reference" "U3"
-			(at 171.45 103.886 0)
+			(at 173.228 78.74 0)
 			(show_name no)
 			(do_not_autoplace no)
@@
 			(project "interfaceBoard"
 				(path "/235e1922-7e9c-45bb-adad-cde682cd8f35/0a67c760-5d0c-4ab0-af6d-0b8dc2801250"
-					(reference "U4")
+					(reference "U9")
 					(unit 1)
 				)
 				(path "/235e1922-7e9c-45bb-adad-cde682cd8f35/ace3e8c2-cc38-4069-a11b-1d2b6aa18c07"
+					(reference "U6")
+					(unit 1)
+				)
+				(path "/235e1922-7e9c-45bb-adad-cde682cd8f35/b05a7146-4f58-4f2b-a2a0-5ebabd023900"
 					(reference "U12")
-					(unit 1)
-				)
-				(path "/235e1922-7e9c-45bb-adad-cde682cd8f35/b05a7146-4f58-4f2b-a2a0-5ebabd023900"
-					(reference "U5")
 					(unit 1)
 				)
@@
 		(dnp no)
 		(fields_autoplaced yes)
-		(property "Reference" "#PWR018"
+		(property "Reference" "#PWR015"
 			(at 157.48 123.19 0)
 			(hide yes)
@@
 			(project "interfaceBoard"
 				(path "/235e1922-7e9c-45bb-adad-cde682cd8f35/0a67c760-5d0c-4ab0-af6d-0b8dc2801250"
+					(reference "#PWR027")
+					(unit 1)
+				)
+				(path "/235e1922-7e9c-45bb-adad-cde682cd8f35/ace3e8c2-cc38-4069-a11b-1d2b6aa18c07"
 					(reference "#PWR021")
 					(unit 1)
 				)
-				(path "/235e1922-7e9c-45bb-adad-cde682cd8f35/ace3e8c2-cc38-4069-a11b-1d2b6aa18c07"
-					(reference "#PWR036")
-					(unit 1)
-				)
 				(path "/235e1922-7e9c-45bb-adad-cde682cd8f35/b05a7146-4f58-4f2b-a2a0-5ebabd023900"
-					(reference "#PWR024")
+					(reference "#PWR033")
 					(unit 1)
 				)
 				(path "/235e1922-7e9c-45bb-adad-cde682cd8f35/b56f998e-c99b-4141-ba0e-9bae5386b37e"
-					(reference "#PWR018")
+					(reference "#PWR015")
 					(unit 1)
 				)
@@
 		(dnp no)
 		(fields_autoplaced yes)
-		(property "Reference" "#PWR019"
+		(property "Reference" "#PWR016"
 			(at 170.18 130.81 0)
 			(hide yes)
@@
 			(project "interfaceBoard"
 				(path "/235e1922-7e9c-45bb-adad-cde682cd8f35/0a67c760-5d0c-4ab0-af6d-0b8dc2801250"
+					(reference "#PWR028")
+					(unit 1)
+				)
+				(path "/235e1922-7e9c-45bb-adad-cde682cd8f35/ace3e8c2-cc38-4069-a11b-1d2b6aa18c07"
 					(reference "#PWR022")
 					(unit 1)
 				)
-				(path "/235e1922-7e9c-45bb-adad-cde682cd8f35/ace3e8c2-cc38-4069-a11b-1d2b6aa18c07"
-					(reference "#PWR037")
-					(unit 1)
-				)
 				(path "/235e1922-7e9c-45bb-adad-cde682cd8f35/b05a7146-4f58-4f2b-a2a0-5ebabd023900"
-					(reference "#PWR025")
+					(reference "#PWR034")
 					(unit 1)
 				)
 				(path "/235e1922-7e9c-45bb-adad-cde682cd8f35/b56f998e-c99b-4141-ba0e-9bae5386b37e"
-					(reference "#PWR019")
+					(reference "#PWR016")
 					(unit 1)
 				)
@@
 			(project "interfaceBoard"
 				(path "/235e1922-7e9c-45bb-adad-cde682cd8f35/0a67c760-5d0c-4ab0-af6d-0b8dc2801250"
+					(reference "RN6")
+					(unit 1)
+				)
+				(path "/235e1922-7e9c-45bb-adad-cde682cd8f35/ace3e8c2-cc38-4069-a11b-1d2b6aa18c07"
 					(reference "RN4")
 					(unit 1)
 				)
-				(path "/235e1922-7e9c-45bb-adad-cde682cd8f35/ace3e8c2-cc38-4069-a11b-1d2b6aa18c07"
+				(path "/235e1922-7e9c-45bb-adad-cde682cd8f35/b05a7146-4f58-4f2b-a2a0-5ebabd023900"
 					(reference "RN8")
-					(unit 1)
-				)
-				(path "/235e1922-7e9c-45bb-adad-cde682cd8f35/b05a7146-4f58-4f2b-a2a0-5ebabd023900"
-					(reference "RN6")
 					(unit 1)
 				)
@@
 			(project "interfaceBoard"
 				(path "/235e1922-7e9c-45bb-adad-cde682cd8f35/0a67c760-5d0c-4ab0-af6d-0b8dc2801250"
+					(reference "RN5")
+					(unit 1)
+				)
+				(path "/235e1922-7e9c-45bb-adad-cde682cd8f35/ace3e8c2-cc38-4069-a11b-1d2b6aa18c07"
 					(reference "RN3")
 					(unit 1)
 				)
-				(path "/235e1922-7e9c-45bb-adad-cde682cd8f35/ace3e8c2-cc38-4069-a11b-1d2b6aa18c07"
+				(path "/235e1922-7e9c-45bb-adad-cde682cd8f35/b05a7146-4f58-4f2b-a2a0-5ebabd023900"
 					(reference "RN7")
-					(unit 1)
-				)
-				(path "/235e1922-7e9c-45bb-adad-cde682cd8f35/b05a7146-4f58-4f2b-a2a0-5ebabd023900"
-					(reference "RN5")
 					(unit 1)
 				)
@@
 		(dnp no)
 		(fields_autoplaced yes)
-		(property "Reference" "#PWR017"
+		(property "Reference" "#PWR014"
 			(at 135.89 110.49 0)
 			(hide yes)
@@
 			(project "interfaceBoard"
 				(path "/235e1922-7e9c-45bb-adad-cde682cd8f35/0a67c760-5d0c-4ab0-af6d-0b8dc2801250"
+					(reference "#PWR026")
+					(unit 1)
+				)
+				(path "/235e1922-7e9c-45bb-adad-cde682cd8f35/ace3e8c2-cc38-4069-a11b-1d2b6aa18c07"
 					(reference "#PWR020")
 					(unit 1)
 				)
-				(path "/235e1922-7e9c-45bb-adad-cde682cd8f35/ace3e8c2-cc38-4069-a11b-1d2b6aa18c07"
-					(reference "#PWR035")
-					(unit 1)
-				)
 				(path "/235e1922-7e9c-45bb-adad-cde682cd8f35/b05a7146-4f58-4f2b-a2a0-5ebabd023900"
-					(reference "#PWR023")
+					(reference "#PWR032")
 					(unit 1)
 				)
 				(path "/235e1922-7e9c-45bb-adad-cde682cd8f35/b56f998e-c99b-4141-ba0e-9bae5386b37e"
-					(reference "#PWR017")
-					(unit 1)
-				)
+					(reference "#PWR014")
+					(unit 1)
+				)

Commit message: WIP
Other:
- added sheet voltageDivider (12v-4vVoltage_Divider.kicad_sch)
Changed lines of the file:
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@@
+		)
+	)
+	(sheet
+		(at 106.68 119.38)
+		(size 12.7 3.81)
+		(exclude_from_sim no)
+		(in_bom yes)
+		(on_board yes)
+		(dnp no)
+		(fields_autoplaced yes)
+		(stroke
+			(width 0.1524)
+			(type solid)
+		)
+		(fill
+			(color 0 0 0 0)
+		)
+		(property "Sheetname" "voltageDivider"
+			(at 106.68 118.6684 0)
+			(show_name no)
+			(do_not_autoplace no)
+			(effects
+				(font
+					(size 1.27 1.27)
+				)
+				(justify left bottom)
+			)
+		)
+		(property "Sheetfile" "12v-4vVoltage_Divider.kicad_sch"
+			(at 106.68 123.7746 0)
+			(show_name no)
+			(do_not_autoplace no)
+			(effects
+				(font
+					(size 1.27 1.27)
+				)
+				(justify left top)
+			)
+		)
+		(instances
+			(project "interfaceBoard"
+				(path "/235e1922-7e9c-45bb-adad-cde682cd8f35/b56f998e-c99b-4141-ba0e-9bae5386b37e"
+					(page "10")
+				)
+			)
 		)
 	)
